File: i7000/i7000.sch (KiCad schematic (older format))
At the start: 71 parts, among them CN01 Conn_02x30_Counter_Clockwise, CN04 Conn_02x30_Counter_Clockwise, CN05 Conn_02x07_Counter_Clockwise

Commit message: wip
Parts:
- added G02, G04, G05: 74LS157, symbol Logic_74xx:74LS157
- added unit 3 of G32
- added unit 1 of G32
Connections:
- net ~GFX_SRAM2_CS: now also G32.10; no longer G32.5
- net ~I8251_CS: now also F04.11 (~CS)
- net at G32.6: now also G10.19 (CE)
- net LS157_S: now reaches G03.1 (S)
- net LS157_S: now also G02.1 (S), G04.1 (S), G05.1 (S), G32.1
- net at G11.19 (CE): now also G32.8
- new net: G32.3, G32.5, G32.9
Other:
- note added: "FOOTPRINT\nNAO POPULADO\nNA PCB DO\nI-7000 G"
- moved on the sheet: E02, E13, E14, E32A, E32B, E32C, E32D, E36B, G03, G06, G10, G11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

Commit message: Not sure what was that, but these changes were sitting here on my local copy since the last time I worked on this schematic drawing effort. I guess it is safer to commit it separately before working on anything else.
Parts:
- removed CN?: Conn_02x07_Counter_Clockwise, symbol Connector:Conn_02x07_Counter_Clockwise
- added E04: 2732, symbol memory:2732
Connections:
- net CN04_20: now also CN04.20 (Pin_20)
- net CN04_41: now also CN04.41 (Pin_41)
- net D0: now also CN01.57 (Pin_57)
- net D1: now also CN01.56 (Pin_56)
- net D2: now also CN01.5 (Pin_5)
- net D3: now also CN01.55 (Pin_55)
- net D4: now also CN01.6 (Pin_6)
- net D5: now also CN01.4 (Pin_4)
- net D6: now also CN01.58 (Pin_58)
- net D7: now also CN01.3 (Pin_3)
- net GND: now also E04.12 (GND)
- net Vcc: now also E04.24 (Vcc)
- net ~EPROM_E renamed ~DRIVE_ROM_E
- new net ~MAINCPU_ROM_E: E04.18 (~E)
- new net ~MAINCPU_ROM_G: E04.20 (~G)
Other:
- moved on the sheet: CN01, CN04, CN05, E02, E03, E13, E14, E32A, E32B, E32C, E32D, E36B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

Commit message: anotando alguns componentes que estavam sem referencias
Parts:
- removed F?: 74LS27, symbol Logic_74xx:74LS27
- removed U?: 74LS157, symbol Logic_74xx:74LS157
- gave numbers to parts that had none: 8
Connections:
- net D0: now also E16.2 (D)
- net D1: now also E17.2 (D)
- net D2: now also E18.2 (D)
- net D3: now also E19.2 (D)
- net D4: now also E20.2 (D)
- net D5: now also E21.2 (D)
- net D6: now also E22.2 (D)
- net D7: now also E23.2 (D)

Commit message: splitting drawing into one schematic per PCB
Parts:
- removed CI01: 2732, symbol memory:2732
- removed CI02: 6116, symbol memory:6116
- removed CI03: WD2793A-PL2, symbol chips_not_yet_available_on_kicad:WD2793
- removed CI06, CI07: 74LS240, symbol Logic_74xx:74LS240
- removed CI09: 74LS38, symbol Logic_74xx:74LS38
- removed CI12: 74LS139, symbol Logic_74xx:74LS139
- removed CI13: 74LS273, symbol Logic_74xx:74LS273
- removed CI14: 74LS138, symbol Logic_74xx:74LS138
- removed CI15: 74LS21, symbol Logic_74xx:74LS21
- removed CI16: 74LS123, symbol Logic_74xx:74LS123
- removed CI17: 74LS244, symbol Logic_74xx:74LS244
- removed CI18: 74LS373, symbol Logic_74xx:74LS373
- removed CI19: 74LS04, symbol Logic_74xx:74LS04
- removed CI20: 74LS14, symbol Logic_74xx:74LS14
- removed CI21: 74LS00, symbol Logic_74xx:74LS00
- removed CN01: Conn_02x30_Counter_Clockwise, symbol Connector:Conn_02x30_Counter_Clockwise
- removed R41: R, symbol device:R
- removed U?: 74LS245, symbol Logic_74xx:74LS245
Other:
- note removed: "/FDC_CS = 0 when:\nA13 == 1\nA11 == 0\nA10 == 0\nCN04_14 == 0\nCN04_42 == 1\nCN04_43 == 1\n"
- note removed: "Floppy Controller"

Commit message: iniciando o posicionamento de componentes da PCB principal
Parts:
- CN04: footprint (none) -> Pin_Headers:Pin_Header_Straight_2x30_Pitch2.54mm
- CN05: footprint (none) -> Pin_Headers:Pin_Header_Straight_2x07_Pitch2.54mm
- E01, E02, F01: footprint (none) -> Housings_DIP:DIP-40_W15.24mm
- E03: footprint DIP-28 -> Housings_DIP:DIP-28_W15.24mm
- E04: footprint (none) -> Housings_DIP:DIP-24_W15.24mm_Socket
- E05, E06, E07, E09, E10, E15, G10, G11: footprint (none) -> Housings_DIP:DIP-20_W7.62mm
- E08, E11, E12, E13, E14, E16, E17, E18, E19, E20, E21, E22, E23, F07, F13, G02, G03, G04, G05, G06: footprint (none) -> Housings_DIP:DIP-16_W7.62mm
- E26, E27, E28, E29, E32, E36, F14, F15, F16, G27, G29, G30, G31, G32, G33: footprint (none) -> Housings_DIP:DIP-14_W7.62mm
- F04: footprint (none) -> Housings_DIP:DIP-28_W15.24mm

Commit message: mais um pedacinho do circuito
Parts:
- added G01: MC6845, Housings_DIP:DIP-40_W15.24mm, symbol motorola:MC6845
- added G09: 74LS273, Housings_DIP:DIP-20_W7.62mm, symbol Logic_74xx:74LS273
- added G13: 74LS244, Housings_DIP:DIP-20_W7.62mm, symbol Logic_74xx:74LS244
- added G14: 2732, Housings_DIP:DIP-24_W15.24mm_Socket, symbol memory:2732
- added G18: 74LS166, Housings_DIP:DIP-16_W7.62mm, symbol Logic_74xx:74LS166
- added unit 2 of G29
- added G34: 74LS32, Housings_DIP:DIP-14_W7.62mm, symbol Logic_74xx:74LS32
- added G35: 74LS08, Housings_DIP:DIP-14_W7.62mm, symbol Logic_74xx:74LS08
- added G36: 74LS86, Housings_DIP:DIP-14_W7.62mm, symbol Logic_74xx:74LS86
Connections:
- net A11: now also G06.13 (I1c)
- net A13: now also G06.14 (I0c)
- net DRAM_OUT0: now also E16.14 (Q)
- net DRAM_OUT1: now also E17.14 (Q)
- net DRAM_OUT2: now also E18.14 (Q)
- net DRAM_OUT3: now also E19.14 (Q)
- net DRAM_OUT4: now also E20.14 (Q)
- net DRAM_OUT5: now also E21.14 (Q)
- net DRAM_OUT6: now also E22.14 (Q)
- net DRAM_OUT7: now also E23.14 (Q)
- net GND: now also G06.6 (I1b), G06.8 (GND), G14.12 (GND), G36.4
- net Vcc: now also G14.24 (Vcc)
- net at G06.3 (I1a): now also G34.6
- new net: G09.12 (Q4), G13.11 (I0b), G14.1 (A7)
- new net: G13.16 (O1a), G14.10 (Q1), G18.3 (B)
- new net: G13.14 (O2a), G14.11 (Q2), G18.4 (C)
- new net: G13.12 (O3a), G14.13 (Q3), G18.5 (D)
- new net: G13.9 (O0b), G14.14 (Q4), G18.10 (E)
- new net: G13.7 (O1b), G14.15 (Q5), G18.11 (F)
- new net: G13.5 (O2b), G14.16 (Q6), G18.12 (G)
- new net: G13.3 (O3b), G14.17 (Q7), G18.14 (H)
- new net: G09.19 (Q7), G13.17 (I3b), G14.19 (A10)
- new net: G09.9 (Q3), G13.8 (I3a), G14.2 (A6)
- new net: G09.16 (Q6), G13.15 (I2b), G14.22 (A9)
- new net: G09.15 (Q5), G13.13 (I1b), G14.23 (A8)
- new net: G09.6 (Q2), G13.6 (I2a), G14.3 (A5)
- new net: G09.5 (Q1), G13.4 (I1a), G14.4 (A4)
- new net: G09.2 (Q0), G13.2 (I0a), G14.5 (A3)
- new net: G13.18 (O0a), G14.9 (Q0), G18.2 (A)
- new net: G34.4, G36.3
- new net: G35.3, G36.1
- new net: G34.3, G36.9
- new net: G35.5, G36.10
- new net RA0: G01.38 (RA0), G14.8 (A0), G29.9
- new net RA1: G01.37 (RA1), G14.7 (A1), G29.10
- new net RA2: G01.36 (RA2), G14.6 (A2), G29.12
- new net RA3: G01.35 (RA3), G34.5
- new net RA4: G01.34 (RA4)
- no-connect marks 8 -> 10
Other:
- note added: "FIXME: The pinout of this symbol does not match its footprint on kicad_pcb"
- note added: "G24.7"
- note added: "G24.9"
- moved on the sheet: E18, E19, E22, E23

Commit message: avanços de ontem
Parts:
- added G28: 74LS74, symbol Logic_74xx:74LS74
- added unit 4 of G30
Connections:
- net at G06.15 (E): now also G27.8 (~Q)
- net at G06.9 (Zd), G30.11: now also G28.13 (~R)
- net at G27.10 (~S): now also G28.1 (~R), G28.10 (~S), G28.4 (~S)
- net ~RESET_OUT_DELAYED: now reaches G27.13 (~R)
- net ~RESET_OUT_DELAYED: now also G30.8
- net ~CHARGEN_ROM_G: now reaches G27.9 (Q)
- net ~CHARGEN_ROM_G: now also G14.20 (~G)
- net RESET_OUT_DELAYED: now reaches CN04.23 (Pin_23)
- net RESET_OUT_DELAYED: now also E29.8, G30.9
- net ~CPU_RESET_OUT: now reaches E09.1 (~Mr), E10.1 (~Mr), E29.10, E29.9
- net at E29.11: now also E01.37 (RESET_OUT)
Other:
- note added: "TODO: C225"
- note added: "pode isso?!"
- moved on the sheet: E28F, E29D, E29E, F07, F13A, F13B, F14A, F14B, F15A, F15B, F16B, G06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

Commit message: update footprints and PCB layout
Parts:
- CN05: footprint Pin_Headers:Pin_Header_Straight_2x07_Pitch2.54mm -> Housings_DIP:DIP-14_W7.62mm_Socket
- G28: footprint (none) -> Housings_DIP:DIP-14_W7.62mm
Connections:
- net A5: now also E04.3 (A5)
Other:
- moved on the sheet: E04, E05, E06, E08, E26B, E27F, E28F
