File: i7000/i7000.sch (KiCad schematic (older format))
At the start: 88 parts, among them CN04 Conn_02x30_Counter_Clockwise, CN05 Conn_02x07_Counter_Clockwise

Commit message: use Package_DIP footprints instead of the older ones called Housings_DIP
Parts:
- CN05: footprint Housings_DIP:DIP-14_W7.62mm_Socket -> Package_DIP:DIP-14_W7.62mm_Socket
- E01, E02, F01, F03, G01: footprint Housings_DIP:DIP-40_W15.24mm -> Package_DIP:DIP-40_W15.24mm
- E03, F04: footprint Housings_DIP:DIP-28_W15.24mm -> Package_DIP:DIP-28_W15.24mm
- E04, G14: footprint Housings_DIP:DIP-24_W15.24mm_Socket -> Package_DIP:DIP-24_W15.24mm_Socket
- E05, E06, E07, E09, E10, E15, G09, G10, G11, G13, G15, G16, G17: footprint Housings_DIP:DIP-20_W7.62mm -> Package_DIP:DIP-20_W7.62mm
- E08, E11, E12, E13, E14, E16, E17, E18, E19, E20, E21, E22, E23, F07, F13, G02, G03, G04, G05, G06, G18, G19, G22, G23, G26: footprint Housings_DIP:DIP-16_W7.62mm -> Package_DIP:DIP-16_W7.62mm
- E26, E27, E28, E29, E32, E36, E38, F14, F15, F16, F20, G27, G28, G29, G30, G31, G32, G33, G34, G35, G36: footprint Housings_DIP:DIP-14_W7.62mm -> Package_DIP:DIP-14_W7.62mm
- F02: footprint Housings_DIP:DIP-24_W15.24mm -> Package_DIP:DIP-24_W15.24mm
- G07, G08: footprint (none) -> Package_DIP:DIP-24_W15.24mm
- G12: footprint (none) -> Package_DIP:DIP-20_W7.62mm
- G20, G21: footprint (none) -> Package_DIP:DIP-16_W7.62mm

Commit message: a few more chips
Parts:
- added F05: ADC0808, Package_DIP:DIP-28_W15.24mm, symbol chips_not_yet_available_on_kicad:ADC0808
- added G37: 74128, Package_DIP:DIP-14_W7.62mm, symbol 74xx_IEEE:74128
- added G38, G39: 74LS00, Package_DIP:DIP-14_W7.62mm, symbol 74xx:74LS00
- added G40, G41: 74S140, Package_DIP:DIP-14_W7.62mm, symbol 74xx_IEEE:74S140
Connections:
- net GND: now also G37.7 (GND), G37.7 (GND), G37.7 (GND), G37.7 (GND)
- net VCC: now also G37.14 (VCC), G37.14 (VCC), G37.14 (VCC), G37.14 (VCC)
- net Vcc: now also G40.14 (Vcc), G40.14 (Vcc), G41.14 (Vcc), G41.14 (Vcc)
- new net Gnd: G40.7 (Gnd), G40.7 (Gnd), G41.7 (Gnd), G41.7 (Gnd)
Other:
- note added: "8-Bit μP Compatible\nA/D Converters\nwith 8-Channel Multiplexer"
Changed lines of the file:
@@
+	1    0    0    -1
+$EndComp
+$Comp
+L 74xx:74LS00 G39
+U 1 1 629515B6
+P 66800 29300
+F 0 "G39" H 66800 29625 50  0000 C CNN
+F 1 "74LS00" H 66800 29534 50  0000 C CNN
+F 2 "Package_DIP:DIP-14_W7.62mm" H 66800 29300 50  0001 C CNN
+F 3 "http://www.ti.com/lit/gpn/sn74ls00" H 66800 29300 50  0001 C CNN
+	1    66800 29300
+	1    0    0    -1
+$EndComp
+$Comp
+L 74xx:74LS00 G39
+U 2 1 62953998
+P 67550 29300
+F 0 "G39" H 67550 29625 50  0000 C CNN
+F 1 "74LS00" H 67550 29534 50  0000 C CNN
+F 2 "Package_DIP:DIP-14_W7.62mm" H 67550 29300 50  0001 C CNN
+F 3 "http://www.ti.com/lit/gpn/sn74ls00" H 67550 29300 50  0001 C CNN
+	2    67550 29300
+	1    0    0    -1
+$EndComp
+$Comp
+L 74xx:74LS00 G39
+U 3 1 62954C7C
+P 66800 29900
+F 0 "G39" H 66800 30225 50  0000 C CNN
+F 1 "74LS00" H 66800 30134 50  0000 C CNN
+F 2 "Package_DIP:DIP-14_W7.62mm" H 66800 29900 50  0001 C CNN
+F 3 "http://www.ti.com/lit/gpn/sn74ls00" H 66800 29900 50  0001 C CNN
+	3    66800 29900
+	1    0    0    -1
+$EndComp
+$Comp
+L 74xx:74LS00 G39
+U 4 1 6295607B
+P 67500 29900
+F 0 "G39" H 67500 30225 50  0000 C CNN
+F 1 "74LS00" H 67500 30134 50  0000 C CNN
+F 2 "Package_DIP:DIP-14_W7.62mm" H 67500 29900 50  0001 C CNN
+F 3 "http://www.ti.com/lit/gpn/sn74ls00" H 67500 29900 50  0001 C CNN
+	4    67500 29900
+	1    0    0    -1
+$EndComp
+$Comp
+L 74xx_IEEE:74S140 G40
+U 1 1 62D58F72
+P 69400 29050
+F 0 "G40" H 69400 29516 50  0000 C CNN
+F 1 "74S140" H 69400 29425 50  0000 C CNN
+F 2 "Package_DIP:DIP-14_W7.62mm" H 69400 29050 50  0001 C CNN
+F 3 "" H 69400 29050 50  0001 C CNN
+	1    69400 29050
+	1    0    0    -1
+$EndComp
+$Comp
+L 74xx_IEEE:74S140 G40
+U 2 1 62D5B6D7
+P 69400 29950
+F 0 "G40" H 69400 30416 50  0000 C CNN
+F 1 "74S140" H 69400 30325 50  0000 C CNN
+F 2 "Package_DIP:DIP-14_W7.62mm" H 69400 29950 50  0001 C CNN
+F 3 "" H 69400 29950 50  0001 C CNN
+	2    69400 29950
+	1    0    0    -1
+$EndComp
+$Comp
+L 74xx_IEEE:74S140 G41
+U 1 1 62F4B621
+P 70650 29050
+F 0 "G41" H 70650 29516 50  0000 C CNN
+F 1 "74S140" H 70650 29425 50  0000 C CNN
+F 2 "Package_DIP:DIP-14_W7.62mm" H 70650 29050 50  0001 C CNN
+F 3 "" H 70650 29050 50  0001 C CNN
+	1    70650 29050
+	1    0    0    -1
+$EndComp
+$Comp
+L 74xx_IEEE:74S140 G41
+U 2 1 62F4B8A7
+P 70650 29950
+F 0 "G41" H 70650 30416 50  0000 C CNN
+F 1 "74S140" H 70650 30325 50  0000 C CNN
+F 2 "Package_DIP:DIP-14_W7.62mm" H 70650 29950 50  0001 C CNN
+F 3 "" H 70650 29950 50  0001 C CNN
+	2    70650 29950
+	1    0    0    -1
+$EndComp
+$Comp
+L 74xx_IEEE:74128 G37
+U 1 1 6304DB0D
+P 72100 29000
+F 0 "G37" H 72100 29466 50  0000 C CNN
+F 1 "74128" H 72100 29375 50  0000 C CNN
+F 2 "Package_DIP:DIP-14_W7.62mm" H 72100 29000 50  0001 C CNN
+F 3 "" H 72100 29000 50  0001 C CNN
+	1    72100 29000
+	1    0    0    -1
+$EndComp
+$Comp
+L 74xx_IEEE:74128 G37
+U 2 1 6314B807
+P 72100 29900
+F 0 "G37" H 72100 30366 50  0000 C CNN
+F 1 "74128" H 72100 30275 50  0000 C CNN
+F 2 "Package_DIP:DIP-14_W7.62mm" H 72100 29900 50  0001 C CNN
+F 3 "" H 72100 29900 50  0001 C CNN
+	2    72100 29900
+	1    0    0    -1
+$EndComp
+$Comp
+L 74xx_IEEE:74128 G37
+U 4 1 6314C58B
+P 73400 29900
+F 0 "G37" H 73400 30366 50  0000 C CNN
+F 1 "74128" H 73400 30275 50  0000 C CNN
+F 2 "Package_DIP:DIP-14_W7.62mm" H 73400 29900 50  0001 C CNN
+F 3 "" H 73400 29900 50  0001 C CNN
+	4    73400 29900
+	1    0    0    -1
+$EndComp
+$Comp
+L 74xx_IEEE:74128 G37
+U 3 1 6314DB32
+P 73350 28950
+F 0 "G37" H 73350 29416 50  0000 C CNN
+F 1 "74128" H 73350 29325 50  0000 C CNN
+F 2 "Package_DIP:DIP-14_W7.62mm" H 73350 28950 50  0001 C CNN
+F 3 "" H 73350 28950 50  0001 C CNN
+	3    73350 28950
+	1    0    0    -1
+$EndComp
+Text Notes 67700 32700 1    50   ~ 0
+8-Bit μP Compatible\nA/D Converters\nwith 8-Channel Multiplexer
+$Comp
+L chips_not_yet_available_on_kicad:ADC0808 F05
+U 1 1 6325599B
+P 67500 32300
+F 0 "F05" H 67150 33450 50  0000 C CNN
+F 1 "ADC0808" V 67400 32050 50  0000 C CNN
+F 2 "Package_DIP:DIP-28_W15.24mm" H 67500 32500 50  0001 C CNN
+F 3 "http://www.ti.com/lit/ds/snas562/snas562.pdf" H 67500 32500 50  0001 C CNN
+	1    67500 32300
+	1    0    0    -1
+$EndComp
+$Comp
+L 74xx:74LS00 G38
+U 1 1 6346C1B2
+P 69450 31300
+F 0 "G38" H 69450 31625 50  0000 C CNN
+F 1 "74LS00" H 69450 31534 50  0000 C CNN
+F 2 "Package_DIP:DIP-14_W7.62mm" H 69450 31300 50  0001 C CNN
+F 3 "http://www.ti.com/lit/gpn/sn74ls00" H 69450 31300 50  0001 C CNN
+	1    69450 31300
+	1    0    0    -1
+$EndComp
+$Comp
+L 74xx:74LS00 G38
+U 2 1 6346C928
+P 70200 31300
+F 0 "G38" H 70200 31625 50  0000 C CNN
+F 1 "74LS00" H 70200 31534 50  0000 C CNN
+F 2 "Package_DIP:DIP-14_W7.62mm" H 70200 31300 50  0001 C CNN
+F 3 "http://www.ti.com/lit/gpn/sn74ls00" H 70200 31300 50  0001 C CNN
+	2    70200 31300
+	1    0    0    -1
+$EndComp
+$Comp
+L 74xx:74LS00 G38
+U 3 1 6346C932
+P 69450 31900
+F 0 "G38" H 69450 32225 50  0000 C CNN
+F 1 "74LS00" H 69450 32134 50  0000 C CNN
+F 2 "Package_DIP:DIP-14_W7.62mm" H 69450 31900 50  0001 C CNN
+F 3 "http://www.ti.com/lit/gpn/sn74ls00" H 69450 31900 50  0001 C CNN
+	3    69450 31900
+	1    0    0    -1
+$EndComp
+$Comp
+L 74xx:74LS00 G38
+U 4 1 6346C93C
+P 70150 31900
+F 0 "G38" H 70150 32225 50  0000 C CNN
+F 1 "74LS00" H 70150 32134 50  0000 C CNN
+F 2 "Package_DIP:DIP-14_W7.62mm" H 70150 31900 50  0001 C CNN
+F 3 "http://www.ti.com/lit/gpn/sn74ls00" H 70150 31900 50  0001 C CNN
+	4    70150 31900
 	1    0    0    -1
 $EndComp

Commit message: coloquei todos os chips no esquemático e na PCB. Agora falta "só" mapear os sinais...
Parts:
- added E24, E25, F08, F11, F12, G25: 74LS74, Package_DIP:DIP-14_W7.62mm, symbol 74xx:74LS74
- added unit 1 of E26
- added E30: 74LS02, Package_DIP:DIP-14_W7.62mm, symbol 74xx:74LS02
- added E31, E34: 74LS08, Package_DIP:DIP-14_W7.62mm, symbol 74xx:74LS08
- added E33: 74LS32, Package_DIP:DIP-14_W7.62mm, symbol 74xx:74LS32
- added E35: 74LS00, Package_DIP:DIP-14_W7.62mm, symbol 74xx:74LS00
- added E37, F22, F23: SN74LS07N, Package_DIP:DIP-14_W7.62mm, symbol 74xx:SN74LS07N
- added F06: 74LS138, Package_DIP:DIP-16_W7.62mm, symbol 74xx:74LS138
- added F10, F9: 74LS163, Package_DIP:DIP-16_W7.62mm, symbol 74xx:74LS163
- added F17: MC1488, Package_DIP:DIP-14_W7.62mm, symbol chips_not_yet_available_on_kicad:MC1488
- added F18, F19: MC1489, Package_DIP:DIP-14_W7.62mm, symbol chips_not_yet_available_on_kicad:MC1489
- added F21: 74LS04, Package_DIP:DIP-14_W7.62mm, symbol 74xx:74LS04
Connections:
- net F17.2_MC1488: no longer names the net of F02.17 (OUT2)
- net F17.2_MC1488: now also F17.2
- net F17.9_MC1488: no longer names the net of F02.13 (OUT1)
- net F17.9_MC1488: now also F17.9
Other:
- moved on the sheet: E27A, F02, F05, G07, G08, G12, G20, G21, G37A, G37B, G37C, G37D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
